File: hardware/Badge_JSCON_2026.kicad_pcb (KiCad board)
At the start: 2 copper layers, 38 parts, among them J2 LCD, P1 USB_C_Plug_USB2.0, Q2 BC846, SW3 ON, U1 ESP32-S3-WROOM-1-N8, U2 BL8072CLTR33, U5 VGdd79S915N0S1

Commit message: feat(Hw):Init_Floorplan
Parts:
- added REF**: Display, Footprints:Display, F.Cu at (176.6, 73.3)
- AE1, C1, C10, C11, C12, C13, C2, C3, C4, C5, C6, C7, C8, C9, F1, J2, P1, Q2, R1, R12, R13, R14, R17, R18, R2, R3, R5, R8, SW1, SW2, SW3, U1, U2, U5: moved to B.Cu
- moved SW2 143.3 mm to (189.5, 118.1)
- moved SW5 132.3 mm to (189.8, 103.4), turned to 180 degrees
- moved SW1 126.3 mm to (165.1, 118.1)
- moved C5 123.6 mm to (194.6, 118.1), turned to 90 degrees
- moved SW6 120.8 mm to (177.3, 111.6), turned to 180 degrees
- moved U5 120.2 mm to (192.2, 42.7)
- moved P1 120.0 mm to (206.5, 93.0), turned to -107 degrees
- moved R5 116.7 mm to (196.0, 118.1), turned to -90 degrees
- moved SW7 115.2 mm to (177.3, 95.2), turned to 180 degrees
- moved F1 114.0 mm to (200.5, 95.0), turned to 180 degrees
- moved R1 112.6 mm to (201.9, 91.2)
- moved R2 111.3 mm to (200.5, 93.6)
- moved SW4 110.8 mm to (164.1, 103.4), turned to 180 degrees
- moved C9 109.1 mm to (189.8, 99.6), turned to 180 degrees
- moved AE1 108.8 mm to (209.8, 45.5), turned to -148 degrees
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Other:
- board outline added: 78.1 x 98.6 mm

Commit message: feat(Hw):Init_Route
Parts:
- removed R17, R18: 4.7K, Resistor_SMD:R_0603_1608Metric
- moved C11 6.40 mm to (172.1, 95.2), turned to 90 degrees
- moved C12 2.54 mm to (186.3, 39.1)
- moved C13 2.54 mm to (184.8, 39.1)
- moved R8 2.54 mm to (184.9, 41.4)
- moved U5 2.54 mm to (194.7, 42.9)
- moved R12 2.54 mm to (184.9, 47.4)
- moved R2 1.37 mm to (201.6, 94.3)
- moved F1 1.36 mm to (201.6, 95.8)
- moved R1 0.88 mm to (202.7, 91.4)
- moved Q2 0.66 mm to (143.9, 74.6)
- moved R13 0.66 mm to (142.2, 77.1)
- moved R14 0.66 mm to (147.6, 74.6)
- moved J2 0.66 mm to (154.1, 73.3)
- moved R3 0.66 mm to (147.6, 72.5)
Connections:
- net /SCL renamed /SPI_SCLK
- net /SDA renamed /SPI_MOSI
- U1 pad 10: /MISO2 -> unconnected-(U1-IO17-Pad10)
- U1 pad 12: /IRQ -> unconnected-(U1-IO8-Pad12)
- U1 pad 22: /CS2 -> unconnected-(U1-IO14-Pad22)
- U1 pad 34: /SCL1 -> unconnected-(U1-IO41-Pad34)
- U1 pad 35: /SDA1 -> unconnected-(U1-IO42-Pad35)
- U1 pad 4: /SDN -> unconnected-(U1-IO4-Pad4)
- U1 pad 5: /IO2 -> unconnected-(U1-IO5-Pad5)
- U1 pad 6: /IO0 -> unconnected-(U1-IO6-Pad6)
- U1 pad 7: /IO1 -> unconnected-(U1-IO7-Pad7)
- U1 pad 8: /SCK2 -> unconnected-(U1-IO15-Pad8)
- U1 pad 9: /MOSI2 -> unconnected-(U1-IO16-Pad9)
Routing:
- net +3.3V: track 0.00 -> 194.7 mm, vias 0 -> 6
- net /EN: track 0.00 -> 119.5 mm, vias 0 -> 2
- net /DOWN: track 0.00 -> 97.6 mm, vias 0 -> 2
- net /BOOT: track 0.00 -> 91.7 mm, vias 0 -> 4
- net /RIGHT: track 0.00 -> 86.3 mm, vias 0 -> 2
- net /LEFT: track 0.00 -> 79.1 mm, vias 0 -> 2
- net /UP: track 0.00 -> 78.5 mm, vias 0 -> 2
- net /D-: track 0.00 -> 77.3 mm
- net /D+: track 0.00 -> 77.2 mm
- net /DIO: track 0.00 -> 62.6 mm, vias 0 -> 2
- net VBUS: track 0.00 -> 57.1 mm
- net /BUSY: track 0.00 -> 54.6 mm, vias 0 -> 2
- net /CS0: track 0.00 -> 47.2 mm, vias 0 -> 2
- net /SCK: track 0.00 -> 44.5 mm, vias 0 -> 2
- net /MISO: track 0.00 -> 43.4 mm, vias 0 -> 2
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- added copper zone on B.Cu, net GND
- added copper zone on F.Cu, net GND

Commit message: feat(Hw):Update_Route
Routing:
- net Net-(F1-Pad1): track 3.02 -> 11.0 mm
- net GND: track 7.14 -> 11.1 mm
- net /D-: track 77.3 -> 80.5 mm
- net /D+: track 77.2 -> 80.2 mm

Commit message: feat(Hw):Update_Route
Routing:
- net +3.3V: track 194.7 -> 201.2 mm, vias 6 -> 14
- net GND: vias 24 -> 33

Commit message: feat(Hw):Update_Labels
Parts:
- added kibuzzard-6A3B0259: G***, kibuzzard-6A3B0259, B.Cu at (165.1, 122.0)
- added kibuzzard-6A3B0260: G***, kibuzzard-6A3B0260, B.Cu at (189.6, 122.1)
- added kibuzzard-6A3B0265: G***, kibuzzard-6A3B0265, B.Cu at (152.4, 103.5)
- added kibuzzard-6A3B026D: G***, kibuzzard-6A3B026D, B.Cu at (151.0, 100.5)
Other:
- board text added: "https://github.com/ElectronicCats/badge_JSCON_2026"
